Commit message: Modifications to support 2+ robots

File: jackal_description/urdf/accessories.urdf.xacro (robot description, xacro)
@@ -1,140 +1,155 @@
 <?xml version="1.0"?>
 <robot xmlns:xacro="http://www.ros.org/wiki/xacro">
-  <!--
-    As you add to this URDF, please be aware that both the robot and
-    simulation include it. You must retain compatibility with all of
-    the following launch files:
-    jackal_viz/launch/view_model.launch
-    jackal_gazebo/launch/jackal_world.launch
-    jackal_base/launch/base.launch
-  -->
-  <!-- Macros to generate standoffs for offset payload mounting. -->
-  <xacro:include filename="$(find jackal_description)/urdf/accessories/standoffs.urdf.xacro" />
-  <!-- This optional plate mounts both the upgraded GPS and the Velodyne 3D LIDAR. -->
-  <xacro:include filename="$(find jackal_description)/urdf/accessories/bridge_plate.urdf.xacro" />
-  <!-- If enabled, generate the LASER payload (by default, a SICK LMS111). -->
-  <xacro:include filename="$(find jackal_description)/urdf/accessories/sick_lms1xx_mount.urdf.xacro" />
-  <xacro:if value="$(optenv JACKAL_LASER 0)">
-    <sick_lms1xx_mount prefix="$(optenv JACKAL_LASER_MOUNT front)"
-                       topic="$(optenv JACKAL_LASER_TOPIC front/scan)"/>
-    <joint name="$(optenv JACKAL_LASER_MOUNT front)_laser_mount_joint" type="fixed">
-      <origin xyz="$(optenv JACKAL_LASER_OFFSET 0 0 0)"
-              rpy="$(optenv JACKAL_LASER_RPY 0 0 0)" />
-      <parent link="$(optenv JACKAL_LASER_MOUNT front)_mount" />
-      <child link="$(optenv JACKAL_LASER_MOUNT front)_laser_mount" />
-    </joint>
-  </xacro:if>
-  <!-- If enabled, generate the upgraded Navsat payload (a Novatel Smart6). -->
-  <xacro:include filename="$(find jackal_description)/urdf/accessories/novatel_smart6.urdf.xacro" />
-  <xacro:if value="$(optenv JACKAL_NAVSAT 0)">
-    <bridge_plate mount="$(optenv JACKAL_NAVSAT_MOUNT rear)"
-                  height="$(optenv JACKAL_NAVSAT_HEIGHT 0.1)" />
-    <novatel_smart6 prefix="$(optenv JACKAL_NAVSAT_MOUNT rear)"/>
-    <joint name="$(optenv JACKAL_NAVSAT_MOUNT rear)_navsat_joint" type="fixed">
-      <origin xyz="0 0 0" rpy="0 0 0" />
-      <parent link="$(optenv JACKAL_NAVSAT_MOUNT rear)_bridge" />
-      <child link="$(optenv JACKAL_NAVSAT_MOUNT rear)_navsat" />
-    </joint>
-  </xacro:if>
-  <!-- Common camera mounts and accessory URDFs. -->
-  <!-- <xacro:include filename="$(find jackal_description)/urdf/accessories/camera_mount.urdf.xacro" /> -->
-  <!-- <xacro:include filename="$(find pointgrey_camera_description)/urdf/pointgrey_flea3.urdf.xacro" /> -->
-  <!-- If enabled, generate the flea3 camera payload with a tilt of 30 degrees. -->
-  <!-- <xacro:if value="$(optenv JACKAL_FLEA3 0)">
-    <camera_mount prefix="$(optenv JACKAL_FLEA3_MOUNT front)"
-                       tilt="$(optenv JACKAL_FLEA3_TILT 0.5236)"/>
-    <joint name="$(optenv JACKAL_FLEA3_MOUNT front)_camera_mount_joint" type="fixed">
-      <origin xyz="$(optenv JACKAL_FLEA3_OFFSET 0 0 0)"
-              rpy="$(optenv JACKAL_FLEA3_RPY 0 0 0)" />
-      <parent link="$(optenv JACKAL_FLEA3_MOUNT front)_mount" />
-      <child link="$(optenv JACKAL_FLEA3_MOUNT front)_camera_mount" />
-    </joint>
-    <pointgrey_flea3 frame="$(optenv JACKAL_FLEA3_MOUNT front)_camera" name="$(optenv JACKAL_FLEA3_NAME front)"
-      camera_x="0.0754" camera_y="0.029" camera_z="0.029"
-      camera_mass="0.085" hfov="1.0471975512" fps="60" width="640" height="512"/>
-    <joint name="$(optenv JACKAL_FLEA3_MOUNT front)_camera_bracket_joint" type="fixed">
-      <origin xyz="0.020 0 0.0245" rpy="0 0 0" />
-      <parent link="$(optenv JACKAL_FLEA3_MOUNT front)_camera_beam" />
-      <child link="$(optenv JACKAL_FLEA3_MOUNT front)_camera" />
-    </joint>
-  </xacro:if> -->
-  <!-- <xacro:include filename="$(find jackal_description)/urdf/accessories/stereo_camera_mount.urdf.xacro" /> -->
-  <!-- If enabled, generates a pair of flea3 cameras for stereo vision with a tilt of 30 degrees. -->
-  <!-- Disabled temporarily due to metapackage issue. -->
-  <!-- <xacro:if value="$(optenv JACKAL_STEREO_FLEA3 0)">
-    <stereo_camera_mount prefix="$(optenv JACKAL_FLEA3_MOUNT front)"
-                       tilt="$(optenv JACKAL_FLEA3_TILT 0.5236)"/>
-    <joint name="$(optenv JACKAL_FLEA3_MOUNT front)_stereo_camera_mount_joint" type="fixed">
-      <origin xyz="$(optenv JACKAL_FLEA3_OFFSET 0 0 0)"
-              rpy="$(optenv JACKAL_FLEA3_RPY 0 0 0)" />
-      <parent link="$(optenv JACKAL_FLEA3_MOUNT front)_mount" />
-      <child link="$(optenv JACKAL_FLEA3_MOUNT front)_stereo_camera_mount" />
-    </joint>
-    <pointgrey_flea3 frame="$(optenv JACKAL_FLEA3_MOUNT front)_left_camera" name="$(optenv JACKAL_FLEA3_LEFT_NAME front/left)"
-      camera_x="0.0754" camera_y="0.029" camera_z="0.029"
-      camera_mass="0.085" hfov="1.0471975512" fps="60" width="640" height="512"/>
-    <joint name="$(optenv JACKAL_FLEA3_MOUNT front)_left_stereo_camera_bracket_joint" type="fixed">
-      <origin xyz="0.015 $(optenv JACKAL_STEREO_SEPERATION 0.16) 0.0599" rpy="0 0 0" />
-      <parent link="$(optenv JACKAL_FLEA3_MOUNT front)_stereo_camera_beam" />
-      <child link="$(optenv JACKAL_FLEA3_MOUNT front)_left_camera" />
-    </joint>
-    <pointgrey_flea3 frame="$(optenv JACKAL_FLEA3_MOUNT front)_right_camera" name="$(optenv JACKAL_FLEA3_RIGHT_NAME front/right)"
-      camera_x="0.0754" camera_y="0.029" camera_z="0.029"
-      camera_mass="0.085" hfov="1.0471975512" fps="60" width="640" height="512"/>
-    <joint name="$(optenv JACKAL_FLEA3_MOUNT front)_right_stereo_camera_bracket_joint" type="fixed">
-      <origin xyz="0.015 -$(optenv JACKAL_STEREO_SEPERATION 0.16) 0.0599" rpy="0 0 0" />
-      <parent link="$(optenv JACKAL_FLEA3_MOUNT front)_stereo_camera_beam" />
-      <child link="$(optenv JACKAL_FLEA3_MOUNT front)_right_camera" />
-    </joint>
-  </xacro:if> -->
-  <!-- If enabled, generate the bumblebee2 camera payload with a tilt of 0 degrees. -->
-  <!-- <xacro:include filename="$(find pointgrey_camera_description)/urdf/pointgrey_bumblebee2.urdf.xacro" /> -->
-  <!-- If enabled, generate the bumblebee2 camera payload with a tilt of 0 degrees. -->
-  <!-- Disabled temporarily due to metapackage issue. -->
-  <!-- <xacro:if value="$(optenv JACKAL_BB2 0)">
-    <camera_mount prefix="$(optenv JACKAL_BB2_MOUNT front)"
-                        tilt="$(optenv JACKAL_BB2_TILT 0)"/>
-    <joint name="$(optenv JACKAL_BB2_MOUNT front)_camera_mount_joint" type="fixed">
-      <origin xyz="$(optenv JACKAL_BB2_OFFSET 0 0 0)"
-              rpy="$(optenv JACKAL_BB2_RPY 0 0 0)" />
-      <parent link="$(optenv JACKAL_BB2_MOUNT front)_mount" />
-      <child link="$(optenv JACKAL_BB2_MOUNT front)_camera_mount" />
-    </joint>
-    <BB2-08S2C-38 frame="$(optenv JACKAL_BB2_MOUNT front)_camera" name="$(optenv JACKAL_BB2_NAME front)" />
-    <joint name="$(optenv JACKAL_BB2_MOUNT front)_camera_bracket_joint" type="fixed">
-      <origin xyz="0.007 0 0.02450" rpy="0 0 0" />
-      <parent link="$(optenv JACKAL_BB2_MOUNT front)_camera_beam" />
-      <child link="$(optenv JACKAL_BB2_MOUNT front)_camera" />
-    </joint>
-  </xacro:if> -->
-  <xacro:include filename="$(find jackal_description)/urdf/accessories/hokuyo_ust10.urdf.xacro" />
-  <xacro:if value="$(optenv JACKAL_FRONT_ACCESSORY_FENDER 0)">
-    <xacro:if value="$(optenv JACKAL_FRONT_FENDER_UST10 0)">
-        <hokuyo_ust10 prefix="front_ust10" parent_link="front_fender_accessory_link"/>
+  <xacro:macro name="jackal_accessories" params="ns">
+    <!--
+      As you add to this URDF, please be aware that both the robot and
+      simulation include it. You must retain compatibility with all of
+      the following launch files:
+      jackal_viz/launch/view_model.launch
+      jackal_gazebo/launch/jackal_world.launch
+      jackal_base/launch/base.launch
+    -->
+    <!-- Macros to generate standoffs for offset payload mounting. -->
+    <xacro:include filename="$(find jackal_description)/urdf/accessories/standoffs.urdf.xacro" />
+    <!-- This optional plate mounts both the upgraded GPS and the Velodyne 3D LIDAR. -->
+    <xacro:include filename="$(find jackal_description)/urdf/accessories/bridge_plate.urdf.xacro" />
+    <!-- If enabled, generate the LASER payload (by default, a SICK LMS111). -->
+    <xacro:include filename="$(find jackal_description)/urdf/accessories/sick_lms1xx_mount.urdf.xacro" />
+    <xacro:if value="$(optenv JACKAL_LASER 0)">
+      <sick_lms1xx_mount prefix="$(optenv JACKAL_LASER_MOUNT front)"
+                         topic="$(optenv JACKAL_LASER_TOPIC front/scan)"/>
+      <joint name="$(optenv JACKAL_LASER_MOUNT front)_laser_mount_joint" type="fixed">
+        <origin xyz="$(optenv JACKAL_LASER_OFFSET 0 0 0)"
+                rpy="$(optenv JACKAL_LASER_RPY 0 0 0)" />
+        <parent link="$(optenv JACKAL_LASER_MOUNT front)_mount" />
+        <child link="$(optenv JACKAL_LASER_MOUNT front)_laser_mount" />
+      </joint>
     </xacro:if>
-  </xacro:if>
-  <xacro:if value="$(optenv JACKAL_REAR_ACCESSORY_FENDER 0)">
-    <xacro:if value="$(optenv JACKAL_REAR_FENDER_UST10 0)">
-        <hokuyo_ust10 prefix="rear_ust10" parent_link="rear_fender_accessory_link"/>
+    <!-- If enabled, generate the LASER payload (by default, a SICK LMS111). -->
+    <xacro:include filename="$(find jackal_description)/urdf/accessories/OS1_mount.urdf.xacro" />
+    <xacro:if value="$(optenv JACKAL_OS1 0)">
+      <OS1_mount prefix="$(optenv JACKAL_LASER_MOUNT front)"
+	      topic="$(optenv JACKAL_LASER_TOPIC front/scan)"
+	      ns="${ns}"/>
+      <joint name="$(optenv JACKAL_LASER_MOUNT front)_laser_mount_joint" type="fixed">
+        <origin xyz="$(optenv JACKAL_LASER_OFFSET 0 0 0)"
+                rpy="$(optenv JACKAL_LASER_RPY 0 0 0)" />
+        <parent link="$(optenv JACKAL_LASER_MOUNT front)_mount" />
+        <child link="$(optenv JACKAL_LASER_MOUNT front)_laser_mount" />
+      </joint>
     </xacro:if>
-  </xacro:if>
-  <xacro:if value="$(optenv JACKAL_ARK_ENCLOSURE 0)">
-    <link name="ark_enclosure_link">
-      <visual>
-        <origin xyz="0 0 0" rpy="0 0 0"/>
-        <geometry>
-          <mesh filename="package://jackal_description/meshes/ark_enclosure.stl"/>
-        </geometry>
-        <material name="dark_grey" />
-      </visual>
-    </link>
-    <joint name="ark_enclosure_joint" type="fixed">
-      <parent link="mid_mount" />
-      <child link="ark_enclosure_link" />
-    </joint>
-    <gazebo reference="ark_enclosure_link">
-      <material>Gazebo/DarkGrey</material>
-      <turnGravityOff>false</turnGravityOff>
-    </gazebo>
-  </xacro:if>
+    <!-- If enabled, generate the upgraded Navsat payload (a Novatel Smart6). -->
+    <xacro:include filename="$(find jackal_description)/urdf/accessories/novatel_smart6.urdf.xacro" />
+    <xacro:if value="$(optenv JACKAL_NAVSAT 0)">
+      <bridge_plate mount="$(optenv JACKAL_NAVSAT_MOUNT rear)"
+                    height="$(optenv JACKAL_NAVSAT_HEIGHT 0.1)" />
+      <novatel_smart6 prefix="$(optenv JACKAL_NAVSAT_MOUNT rear)"/>
+      <joint name="$(optenv JACKAL_NAVSAT_MOUNT rear)_navsat_joint" type="fixed">
+        <origin xyz="0 0 0" rpy="0 0 0" />
+        <parent link="$(optenv JACKAL_NAVSAT_MOUNT rear)_bridge" />
+        <child link="$(optenv JACKAL_NAVSAT_MOUNT rear)_navsat" />
+      </joint>
+    </xacro:if>
+    <!-- Common camera mounts and accessory URDFs. -->
+    <!-- <xacro:include filename="$(find jackal_description)/urdf/accessories/camera_mount.urdf.xacro" /> -->
+    <!-- <xacro:include filename="$(find pointgrey_camera_description)/urdf/pointgrey_flea3.urdf.xacro" /> -->
+    <!-- If enabled, generate the flea3 camera payload with a tilt of 30 degrees. -->
+    <!-- <xacro:if value="$(optenv JACKAL_FLEA3 0)">
+      <camera_mount prefix="$(optenv JACKAL_FLEA3_MOUNT front)"
+                         tilt="$(optenv JACKAL_FLEA3_TILT 0.5236)"/>
+      <joint name="$(optenv JACKAL_FLEA3_MOUNT front)_camera_mount_joint" type="fixed">
+        <origin xyz="$(optenv JACKAL_FLEA3_OFFSET 0 0 0)"
+                rpy="$(optenv JACKAL_FLEA3_RPY 0 0 0)" />
+        <parent link="$(optenv JACKAL_FLEA3_MOUNT front)_mount" />
+        <child link="$(optenv JACKAL_FLEA3_MOUNT front)_camera_mount" />
+      </joint>
+      <pointgrey_flea3 frame="$(optenv JACKAL_FLEA3_MOUNT front)_camera" name="$(optenv JACKAL_FLEA3_NAME front)"
+        camera_x="0.0754" camera_y="0.029" camera_z="0.029"
+        camera_mass="0.085" hfov="1.0471975512" fps="60" width="640" height="512"/>
+      <joint name="$(optenv JACKAL_FLEA3_MOUNT front)_camera_bracket_joint" type="fixed">
+        <origin xyz="0.020 0 0.0245" rpy="0 0 0" />
+        <parent link="$(optenv JACKAL_FLEA3_MOUNT front)_camera_beam" />
+        <child link="$(optenv JACKAL_FLEA3_MOUNT front)_camera" />
+      </joint>
+    </xacro:if> -->
+    <!-- <xacro:include filename="$(find jackal_description)/urdf/accessories/stereo_camera_mount.urdf.xacro" /> -->
+    <!-- If enabled, generates a pair of flea3 cameras for stereo vision with a tilt of 30 degrees. -->
+    <!-- Disabled temporarily due to metapackage issue. -->
+    <!-- <xacro:if value="$(optenv JACKAL_STEREO_FLEA3 0)">
+      <stereo_camera_mount prefix="$(optenv JACKAL_FLEA3_MOUNT front)"
+                         tilt="$(optenv JACKAL_FLEA3_TILT 0.5236)"/>
+      <joint name="$(optenv JACKAL_FLEA3_MOUNT front)_stereo_camera_mount_joint" type="fixed">
+        <origin xyz="$(optenv JACKAL_FLEA3_OFFSET 0 0 0)"
+                rpy="$(optenv JACKAL_FLEA3_RPY 0 0 0)" />
+        <parent link="$(optenv JACKAL_FLEA3_MOUNT front)_mount" />
+        <child link="$(optenv JACKAL_FLEA3_MOUNT front)_stereo_camera_mount" />
+      </joint>
+      <pointgrey_flea3 frame="$(optenv JACKAL_FLEA3_MOUNT front)_left_camera" name="$(optenv JACKAL_FLEA3_LEFT_NAME front/left)"
+        camera_x="0.0754" camera_y="0.029" camera_z="0.029"
+        camera_mass="0.085" hfov="1.0471975512" fps="60" width="640" height="512"/>
+      <joint name="$(optenv JACKAL_FLEA3_MOUNT front)_left_stereo_camera_bracket_joint" type="fixed">
+        <origin xyz="0.015 $(optenv JACKAL_STEREO_SEPERATION 0.16) 0.0599" rpy="0 0 0" />
+        <parent link="$(optenv JACKAL_FLEA3_MOUNT front)_stereo_camera_beam" />
+        <child link="$(optenv JACKAL_FLEA3_MOUNT front)_left_camera" />
+      </joint>
+      <pointgrey_flea3 frame="$(optenv JACKAL_FLEA3_MOUNT front)_right_camera" name="$(optenv JACKAL_FLEA3_RIGHT_NAME front/right)"
+        camera_x="0.0754" camera_y="0.029" camera_z="0.029"
+        camera_mass="0.085" hfov="1.0471975512" fps="60" width="640" height="512"/>
+      <joint name="$(optenv JACKAL_FLEA3_MOUNT front)_right_stereo_camera_bracket_joint" type="fixed">
+        <origin xyz="0.015 -$(optenv JACKAL_STEREO_SEPERATION 0.16) 0.0599" rpy="0 0 0" />
+        <parent link="$(optenv JACKAL_FLEA3_MOUNT front)_stereo_camera_beam" />
+        <child link="$(optenv JACKAL_FLEA3_MOUNT front)_right_camera" />
+      </joint>
+    </xacro:if> -->
+    <!-- If enabled, generate the bumblebee2 camera payload with a tilt of 0 degrees. -->
+    <!-- <xacro:include filename="$(find pointgrey_camera_description)/urdf/pointgrey_bumblebee2.urdf.xacro" /> -->
+    <!-- If enabled, generate the bumblebee2 camera payload with a tilt of 0 degrees. -->
+    <!-- Disabled temporarily due to metapackage issue. -->
+    <!-- <xacro:if value="$(optenv JACKAL_BB2 0)">
+      <camera_mount prefix="$(optenv JACKAL_BB2_MOUNT front)"
+                          tilt="$(optenv JACKAL_BB2_TILT 0)"/>
+      <joint name="$(optenv JACKAL_BB2_MOUNT front)_camera_mount_joint" type="fixed">
+        <origin xyz="$(optenv JACKAL_BB2_OFFSET 0 0 0)"
+                rpy="$(optenv JACKAL_BB2_RPY 0 0 0)" />
+        <parent link="$(optenv JACKAL_BB2_MOUNT front)_mount" />
+        <child link="$(optenv JACKAL_BB2_MOUNT front)_camera_mount" />
+      </joint>
+      <BB2-08S2C-38 frame="$(optenv JACKAL_BB2_MOUNT front)_camera" name="$(optenv JACKAL_BB2_NAME front)" />
+      <joint name="$(optenv JACKAL_BB2_MOUNT front)_camera_bracket_joint" type="fixed">
+        <origin xyz="0.007 0 0.02450" rpy="0 0 0" />
+        <parent link="$(optenv JACKAL_BB2_MOUNT front)_camera_beam" />
+        <child link="$(optenv JACKAL_BB2_MOUNT front)_camera" />
+      </joint>
+    </xacro:if> -->
+    <xacro:include filename="$(find jackal_description)/urdf/accessories/hokuyo_ust10.urdf.xacro" />
+    <xacro:if value="$(optenv JACKAL_FRONT_ACCESSORY_FENDER 0)">
+      <xacro:if value="$(optenv JACKAL_FRONT_FENDER_UST10 0)">
+          <hokuyo_ust10 prefix="front_ust10" parent_link="front_fender_accessory_link"/>
+      </xacro:if>
+    </xacro:if>
+    <xacro:if value="$(optenv JACKAL_REAR_ACCESSORY_FENDER 0)">
+      <xacro:if value="$(optenv JACKAL_REAR_FENDER_UST10 0)">
+          <hokuyo_ust10 prefix="rear_ust10" parent_link="rear_fender_accessory_link"/>
+      </xacro:if>
+    </xacro:if>
+    <xacro:if value="$(optenv JACKAL_ARK_ENCLOSURE 0)">
+      <link name="ark_enclosure_link">
+        <visual>
+          <origin xyz="0 0 0" rpy="0 0 0"/>
+          <geometry>
+            <mesh filename="package://jackal_description/meshes/ark_enclosure.stl"/>
+          </geometry>
+          <material name="dark_grey" />
+        </visual>
+      </link>
+      <joint name="ark_enclosure_joint" type="fixed">
+        <parent link="mid_mount" />
+        <child link="ark_enclosure_link" />
+      </joint>
+      <gazebo reference="ark_enclosure_link">
+        <material>Gazebo/DarkGrey</material>
+        <turnGravityOff>false</turnGravityOff>
+      </gazebo>
+    </xacro:if>
+  </xacro:macro>
 </robot>

File: jackal_description/urdf/jackal.urdf.xacro (robot description, xacro)
@@ -2,4 +2,6 @@
 <robot name="jackal" xmlns:xacro="http://www.ros.org/wiki/xacro">
   <xacro:property name="PI" value="3.1415926535897931" />
+  <xacro:property name="namespace" value="jackal" />
+  <xacro:arg name="ns" default="jackal" />
   <xacro:property name="wheelbase" value="0.262" />
   <xacro:property name="track" value="0.37559" />
@@ -223,8 +225,10 @@
   <!-- Bring in simulation data for Gazebo. -->
   <xacro:include filename="$(find jackal_description)/urdf/jackal.gazebo" />
+  <xacro:jackal_gazebo ns="$(arg ns)"/>
   <!-- Optional standard accessories, including their simulation data. The rendering
        of these into the final description is controlled by optenv variables, which
        default each one to off.-->
   <xacro:include filename="$(find jackal_description)/urdf/accessories.urdf.xacro" />
+  <xacro:jackal_accessories ns="$(arg ns)"/>
   <!-- Optional custom includes. -->
   <xacro:include filename="$(optenv JACKAL_URDF_EXTRAS empty.urdf)" />
